File: Keyboard - 100 Key Custom.kicad_pcb (KiCad board)
At the start: 2 copper layers, 363.5 x 115.9 mm, 223 parts, among them J1 TYPE-C-31-M12_13, K1 Esc, K10 A, K100 P_+, K101 P_Enter_200v, K11 Z, K12 Win_L_125, K13 F2, K14 2(@), K15 W, K16 S, K17 X, K18 Alt_L_125, K19 F3, K2 `(~~), K20 3(#), K21 E, K22 D, K23 C, K24 F4, K25 4($), K26 R, K27 F, K28 V, K29 F5, K3 Tab_150, K30 5(%), K31 T, K32 G, K33 B, K34 Space_625, K35 F6, K36 6(^), K37 Y, K38 H, K39 N, K4 Caps_Lock_175, K40 F7, K41 7(&), K42 U, K43 J, K44 M, K45 F8, K46 8(*), K47 I, K48 K, K49 ,(<), K5 Shift_L_225, K50 F9, K51 9((), K52 O, K53 L, K54 .(>), K55 Alt_R, K56 F10, K57 0()), K58 P, K59 ;(:), K6 Ctrl_L_125, K60 /(?), K61 Function, K62 F11, K63 -(_), K64 [({), K65 '("), K66 Ctrl_R, K67 F12, K68 =(+), K69 ](}), K7 F1, K70 Shift_R_175, K71 Left, K72 Print_Screen, K73 Backspace_200, K74 \(|)_150, K75 Enter_225, K76 Up, K77 Down, K78 Delete, K79 Insert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

Commit message: Started tracing
Parts:
- removed D102: PRTR5V0U2X, Package_TO_SOT_SMD:SOT-143
- removed F1: 500mA, Fuse:Fuse_0805_2012Metric_Pad1.15x1.40mm_HandSolder
- removed R1, R2: 5.1k, Capacitor_SMD:C_1206_3216Metric_Pad1.42x1.75mm_HandSolder
- J1: value TYPE-C-31-M12_13 -> SM04B_SRSS; footprint acheronLibrary Connectors:TYPE-C-31-M-12 -> acheronLibrary Connectors:SM04B-SRSS
- moved R5 64.8 mm to (202.9, 69.6), turned to 90 degrees
- moved J1 53.5 mm to (196.9, 70.1)
- moved R6 52.5 mm to (190.8, 69.6), turned to 90 degrees
- moved R3 49.9 mm to (206.5, 87.4), turned to 90 degrees
- moved R4 44.9 mm to (196.1, 87.4), turned to -90 degrees
- moved SW1 44.6 mm to (201.5, 87.6), turned to -90 degrees
- moved C1 43.9 mm to (201.7, 93.2), turned to 0 degrees
- moved C3 30.9 mm to (185.9, 111.8), turned to 0 degrees
- moved C2 27.5 mm to (185.9, 124.0), turned to 0 degrees
- moved C7 14.4 mm to (158.2, 118.4), turned to -90 degrees
- moved U1 12.1 mm to (173.8, 118.1), turned to -90 degrees
- moved C4 11.5 mm to (163.1, 113.8), turned to 0 degrees
- moved R7 10.5 mm to (163.3, 123.7), turned to 0 degrees
- moved C5 10.1 mm to (163.3, 118.4), turned to -90 degrees
- moved Y1 8.61 mm to (185.9, 117.9), turned to -90 degrees
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Routing:
- net row1: track 0.00 -> 369.7 mm
- net row0: track 0.00 -> 369.1 mm
- net col1: track 0.00 -> 112.4 mm
- net col2: track 0.00 -> 110.0 mm
- net col13: track 0.00 -> 109.1 mm
- net col9: track 0.00 -> 107.1 mm
- net col10: track 0.00 -> 107.1 mm
- net col5: track 0.00 -> 106.1 mm
- net col0: track 0.00 -> 104.1 mm
- net col12: track 0.00 -> 103.1 mm
- net col11: track 0.00 -> 103.1 mm
- net col17: track 0.00 -> 95.2 mm
- net col16: track 0.00 -> 95.2 mm
- net col15: track 0.00 -> 95.2 mm
- net col8: track 0.00 -> 86.1 mm
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
Commit message: Removed traces and changed MCU package & footprint
Parts:
- U1: footprint Package_QFP:TQFP-44_10x10mm_P0.8mm -> acheronLibrary Components:QFN-44-1EP_7x7mm_P0.5mm_EP5.2x5.2mm
- moved C1 161.0 mm to (42.2, 71.6)
- moved R4 160.8 mm to (36.6, 67.3)
- moved R3 160.8 mm to (47.0, 67.3)
- moved SW1 152.3 mm to (53.8, 50.3)
- moved R5 136.0 mm to (67.5, 57.1), turned to 0 degrees
- moved U1 133.4 mm to (45.9, 80.4), turned to 0 degrees
- moved J1 125.1 mm to (73.1, 51.8)
- moved R6 124.2 mm to (67.5, 53.8), turned to 0 degrees
- moved C8 23.6 mm to (177.8, 127.3), turned to 180 degrees
- moved C7 18.1 mm to (174.0, 109.5), turned to 0 degrees
- moved C4 7.69 mm to (169.4, 109.5)
- moved C5 4.22 mm to (165.1, 114.5), turned to 90 degrees
- moved C6 3.46 mm to (163.6, 120.4)
- moved R7 2.14 mm to (163.8, 125.8), turned to -90 degrees
Routing:
- net row1: track 369.7 -> 0.00 mm
- net row0: track 369.1 -> 0.00 mm
- net col1: track 112.4 -> 0.00 mm
- net col2: track 110.0 -> 0.00 mm
- net col13: track 109.1 -> 0.00 mm
- net col9: track 107.1 -> 0.00 mm
- net col10: track 107.1 -> 0.00 mm
- net col5: track 106.1 -> 0.00 mm
- net col0: track 104.1 -> 0.00 mm
- net col12: track 103.1 -> 0.00 mm
- net col11: track 103.1 -> 0.00 mm
- net col17: track 95.2 -> 0.00 mm
- net col16: track 95.2 -> 0.00 mm
- net col15: track 95.2 -> 0.00 mm
- net col8: track 86.1 -> 0.00 mm
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Other:
- net class Default: trace_width 0.25 -> 0.254
- net class Power added: clearance 0.2, trace_width 0.381, via_dia 0.8, via_drill 0.4

Commit message: Placed components roughly and traced rows and columns.
Parts:
- moved C2 165.9 mm to (29.7, 68.1), turned to 90 degrees
- moved C3 160.8 mm to (29.7, 73.6), turned to -90 degrees
- moved Y1 159.5 mm to (33.5, 70.8), turned to 90 degrees
- moved C8 142.8 mm to (42.9, 80.3), turned to 0 degrees
- moved C7 142.1 mm to (39.3, 64.2)
- moved C6 129.0 mm to (47.0, 65.3), turned to 135 degrees
- moved C5 124.7 mm to (47.2, 74.0), turned to -135 degrees
- moved C4 117.2 mm to (60.2, 67.1), turned to 180 degrees
- moved R7 114.9 mm to (64.0, 68.8)
- moved J1 19.5 mm to (78.7, 70.6), turned to -90 degrees
- moved R3 17.8 mm to (46.8, 49.5), turned to 0 degrees
- moved R4 17.4 mm to (41.2, 50.5), turned to 180 degrees
- moved R6 16.7 mm to (73.7, 69.3)
- moved R5 15.9 mm to (73.7, 71.8)
- moved U1 10.6 mm to (41.6, 70.7), turned to 90 degrees
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Connections:
- J1 pad 1: VCC -> +5V
Routing:
- net row1: track 0.00 -> 344.8 mm
- net row0: track 0.00 -> 342.9 mm
- net row2: track 0.00 -> 338.1 mm
- net row4: track 0.00 -> 336.6 mm
- net row5: track 0.00 -> 325.7 mm
- net row3: track 0.00 -> 311.6 mm
- net col1: track 0.00 -> 112.4 mm
- net col2: track 0.00 -> 110.0 mm
- net col13: track 0.00 -> 109.1 mm
- net col9: track 0.00 -> 107.1 mm
- net col10: track 0.00 -> 107.1 mm
- net col5: track 0.00 -> 106.1 mm
- net col0: track 0.00 -> 104.1 mm
- net col12: track 0.00 -> 103.1 mm
- net col11: track 0.00 -> 103.1 mm
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Other:
- net class Power: trace_width 0.381 -> 0.3429

Commit message: Added traces besides rows/columns
Parts:
- moved C2 163.4 mm to (186.6, 113.7), turned to -90 degrees
- moved C3 160.7 mm to (186.6, 108.2), turned to 90 degrees
- moved Y1 154.4 mm to (182.6, 110.9), turned to -90 degrees
- moved C7 146.8 mm to (176.2, 117.2), turned to -135 degrees
- moved R3 145.5 mm to (187.3, 87.6), turned to 90 degrees
- moved C1 142.1 mm to (182.6, 89.3), turned to 0 degrees
- moved R4 141.4 mm to (177.6, 87.6), turned to -90 degrees
- moved U1 137.1 mm to (172.7, 111.2), turned to -90 degrees
- moved SW1 133.9 mm to (182.5, 83.1), turned to -90 degrees
- moved C8 132.9 mm to (173.8, 103.5), turned to -90 degrees
- moved C6 128.9 mm to (165.7, 115.4), turned to -45 degrees
- moved C5 123.5 mm to (166.1, 107.4), turned to 45 degrees
- moved C4 117.5 mm to (173.4, 98.7), turned to -90 degrees
- moved R7 111.4 mm to (164.1, 117.6), turned to -45 degrees
- moved R5 91.6 mm to (164.6, 83.1), turned to 90 degrees
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Connections:
- U1 pad 1: Net-(U1-Pad1) -> row4
- U1 pad 41: Net-(U1-Pad41) -> row5
Routing:
- net +5V: track 7.61 -> 114.3 mm, vias 0 -> 7
- net GND: track 11.0 -> 114.1 mm
- net row5: track 325.7 -> 272.4 mm
- net RESET: track 0.00 -> 36.9 mm, vias 0 -> 2
- net row3: track 311.6 -> 337.8 mm
- net Net-(R5-Pad1): track 4.50 -> 27.1 mm, vias 1 -> 0
- net Net-(R6-Pad1): track 4.53 -> 27.1 mm, vias 1 -> 0
- net row4: track 336.6 -> 351.7 mm, vias 0 -> 3
- net Net-(C4-Pad2): track 0.00 -> 8.45 mm
- net Net-(R7-Pad2): track 0.00 -> 7.15 mm
- net Net-(D101-Pad2): track 0.00 -> 4.00 mm
- net Net-(D38-Pad2): track 0.00 -> 3.67 mm
- net Net-(D12-Pad2): track 0.00 -> 3.42 mm
- net Net-(D18-Pad2): track 0.00 -> 3.41 mm
- net Net-(D34-Pad2): track 0.00 -> 3.41 mm
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Other:
- net class Power: trace_width 0.3429 -> 0.29845

Commit message: Replaced MCU with hand-solder model and retraced.
Parts:
- U1: footprint acheronLibrary Components:QFN-44-1EP_7x7mm_P0.5mm_EP5.2x5.2mm -> acheronLibrary Components:TQPF-44_10x10mm_P0.8mm
- moved C7 5.57 mm to (178.3, 122.3)
- moved Y1 4.32 mm to (186.6, 112.6)
- moved C2 4.32 mm to (190.6, 115.4)
- moved C3 4.32 mm to (190.6, 109.9)
- moved R7 3.93 mm to (161.3, 120.4)
- moved C6 3.46 mm to (163.4, 117.9)
- moved C5 2.76 mm to (163.4, 107.9)
- moved C8 2.43 mm to (174.9, 101.4)
- moved U1 1.87 mm to (173.0, 113.0)
- moved C4 1.38 mm to (173.5, 97.3)
Connections:
- U1 pad 1: row4 -> Net-(U1-Pad1)
- U1 pad 41: row5 -> Net-(U1-Pad41)
Routing:
- net +5V: track 114.3 -> 134.5 mm, vias 7 -> 8
- net row5: track 272.4 -> 254.2 mm
- net row4: track 351.7 -> 336.6 mm, vias 3 -> 2
- net GND: track 114.1 -> 128.4 mm
- net Net-(R3-Pad2): track 2.91 -> 9.11 mm
- net Net-(D90-Pad2): track 0.00 -> 3.41 mm
- net Net-(D61-Pad2): track 0.00 -> 3.41 mm
- net Net-(D71-Pad2): track 0.00 -> 3.41 mm
- net Net-(D66-Pad2): track 0.00 -> 3.41 mm
- net Net-(D55-Pad2): track 0.00 -> 3.41 mm
- net Net-(D96-Pad2): track 0.00 -> 3.41 mm
- net Net-(D84-Pad2): track 0.00 -> 3.40 mm
- net Net-(D77-Pad2): track 0.00 -> 3.40 mm
- net RESET: track 36.9 -> 39.8 mm
- net Net-(R7-Pad2): track 7.15 -> 8.60 mm
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Other:
- net class Power: trace_width 0.29845 -> 0.381

Commit message: Finished Running Traces
Parts:
- added HOLE: H**, acheronLibrary Mounting Holes:MountingHole_2.5x5.0mm, F.Cu at (149.3, 32.8)
- added HOLE: H**, acheronLibrary Mounting Holes:MountingHole_2.5x5.0mm, F.Cu at (245.8, 32.8)
- added HOLE: H**, acheronLibrary Mounting Holes:MountingHole_2.5x5.0mm, F.Cu at (254.0, 98.0)
- added HOLE: H**, acheronLibrary Mounting Holes:MountingHole_2.5x5.0mm, F.Cu at (135.0, 105.8)
- added HOLE: H**, acheronLibrary Mounting Holes:MountingHole_2.5x5.0mm, F.Cu at (339.8, 106.7)
- added HOLE: H**, acheronLibrary Mounting Holes:MountingHole_2.5x5.0mm, F.Cu at (339.6, 33.0)
- added HOLE: H**, acheronLibrary Mounting Holes:MountingHole_2.5x5.0mm, F.Cu at (55.5, 101.8)
- added HOLE: H**, acheronLibrary Mounting Holes:MountingHole_2.5x5.0mm, F.Cu at (55.4, 33.0)
- moved C2 2.29 mm to (192.9, 115.4)
- moved C3 2.29 mm to (192.9, 109.9)
- moved Y1 2.29 mm to (188.9, 112.6)
- moved C8 0.63 mm to (174.2, 101.4)
Connections:
- U1 pad 1: Net-(U1-Pad1) -> row4
- U1 pad 10: Net-(U1-Pad10) -> col9
- U1 pad 11: Net-(U1-Pad11) -> col10
- U1 pad 12: Net-(U1-Pad12) -> col11
- U1 pad 18: Net-(U1-Pad18) -> col12
- U1 pad 19: Net-(U1-Pad19) -> col13
- U1 pad 20: Net-(U1-Pad20) -> col14
- U1 pad 21: Net-(U1-Pad21) -> col15
- U1 pad 22: Net-(U1-Pad22) -> col16
- U1 pad 25: Net-(U1-Pad25) -> col17
- U1 pad 26: Net-(U1-Pad26) -> col18
- U1 pad 27: Net-(U1-Pad27) -> col0
- U1 pad 28: Net-(U1-Pad28) -> col1
- U1 pad 29: Net-(U1-Pad29) -> col2
- U1 pad 30: Net-(U1-Pad30) -> col3
- U1 pad 31: Net-(U1-Pad31) -> col4
- U1 pad 32: Net-(U1-Pad32) -> col5
- U1 pad 36: Net-(U1-Pad36) -> col6
- U1 pad 37: Net-(U1-Pad37) -> row0
- U1 pad 38: Net-(U1-Pad38) -> row1
- U1 pad 39: Net-(U1-Pad39) -> row2
- U1 pad 40: Net-(U1-Pad40) -> row3
- U1 pad 41: Net-(U1-Pad41) -> row5
- U1 pad 8: Net-(U1-Pad8) -> col7
- U1 pad 9: Net-(U1-Pad9) -> col8
Routing:
- net row0: track 342.9 -> 608.5 mm
- net row1: track 344.8 -> 588.0 mm
- net row2: track 338.1 -> 565.5 mm
- net col14: track 0.00 -> 220.1 mm, vias 0 -> 3
- net row3: track 337.8 -> 546.3 mm
- net col18: track 85.7 -> 290.7 mm
- net col17: track 95.2 -> 274.0 mm
- net col0: track 104.1 -> 270.6 mm, vias 0 -> 1
- net col16: track 95.2 -> 259.9 mm, vias 0 -> 2
- net col15: track 95.2 -> 239.8 mm, vias 0 -> 2
- net col1: track 112.4 -> 253.5 mm, vias 0 -> 1
- net col13: track 109.1 -> 232.7 mm, vias 0 -> 2
- net col2: track 110.0 -> 224.7 mm, vias 0 -> 1
- net row5: track 254.2 -> 360.7 mm, vias 0 -> 2
- net col3: track 86.1 -> 186.7 mm, vias 0 -> 1
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- added copper zone on B.Cu, net GND

Commit message: Created Gerber Files
Routing:
- net GND: track 108.7 -> 113.1 mm
Other:
- board text added: "I don't know what I'm doing."
- board text added: "KRKB - v1.0"
